Commit message: feat(robot+comm): 串口热重连、零点/URDF 对齐、多键位一键动作与 Jacobian 符号修正
.git / 仓库卫生
- 根 .gitignore：忽略 *.zip、*_Old.STL，避免大体积压缩包与旧网格进入历史。
- 从索引移除 src/TRoMaC_2026_Manipulator.zip（本地可保留作备份；此前误纳入会导致仓库膨胀）。

Serial（TRoMaC::Uart）
- Open()：重连/重开时重置 RX 状态机与环形缓冲，避免半帧残留污染新会话。
- ReadData：select 就绪但 read()<=0 时置 last_read_disconnected_，区分「无数据」与「设备掉线」。
- send：fd 未打开时静默返回，避免 write(-1) 刷屏；open 失败时减少 perror 噪声（重连循环场景）。
- 默认设备映射：comport 1→/dev/ttyUSB0，comport 2→/dev/ttyACM0（与常见 USB 转串口命名对调）。

tromac_hardware_interface
- JOINT_OFFSET_RAD 与 serial_comm_node 中 joint_offset_rad_ 对齐，并补充
  「ros_rad = JOINT_DIR·raw·π/180 + OFFSET」及 J1 人为零点说明。
- on_configure：首次 Open 失败不再 FATAL 退出，交由 readLoop 每 1s 重连，下位机晚
  上电也可先 launch。
- readLoop：未连接时 attemptReconnect；连接后 onReconnectedTriggerSync：等首帧
  RX → 向 /serial_recv 发 Btn=0 合成帧再模拟 Btn=17 上升沿，复用 handleRxFrame
  触发 snapshot + force-sync + serial_comm_node 侧 JTC 重同步，避免重连后 cmd 突跳。
- 断开路径：last_read_disconnected_、select 错误、Close 后 serial_connected_=false。
- write：未连接时丢弃 TX 并 5s 节流告警计数。
- RX 解析与 /serial_recv 发布抽成 handleRxFrame，供正常循环与重连同步共用。

serial_comm_node
- 控制模式：遥控器键位重映射（9/12 前三/后三关节；13 Homing；14/11/10 三套
  GetEnerge_* 预设位姿）；homing_active_ 泛化为 plan_active_，一键动作互斥。
- executeJointTarget：统一 pause_servo → MoveGroup 规划/执行 → stop/start_servo；
  Homing/GetEnerge_1/2/3 仅绑定目标数组与标签；规划成功打 PLAN diag（点数、
  时长、max|vel|）；MoveGroup scale 恢复 1.0。
- 更新 home_target_rad_ 与各 GetEnerge 关节目标常量；Jacobian 笛卡尔 vz 与
  JointJog 第 2 轴速度符号修正（与实机方向一致）。
- 去掉文件头「精简版」说明块（职责仍以代码为准）。

MoveIt / Servo 配置
- joint_limits.yaml：默认速度/加速度缩放 0.1→0.5。
- servo_settings.yaml：linear/rotational/joint scale 1.0→1.50。

manipulator 模型
- manipulator.urdf：1-joint、4-joint 由 continuous 改为带 limit 的 revolute；
  各关节 effort/velocity 写入合理非零值（含 velocity 1.5）。
- meshes/6Link.STL：更新末端连杆网格。

未纳入版本库：符合 .gitignore 的本地 *.zip、6Link_Old.STL（若存在）。

Co-authored-by: Cursor <cursoragent@cursor.com>

File: src/manipulator/urdf/manipulator.urdf (robot description, URDF)
Before this commit: robot manipulator, 7 links, 6 joints
Joints:
- joint 1-joint: limit (none) -> lower=-2.1765 upper=1.1728 effort=27 velocity=1.5; type continuous -> revolute
- joint 2-joint: limit lower=0 upper=2.6834 effort=0 velocity=0 -> lower=0 upper=2.6834 effort=40 velocity=1.5
- joint 3-joint: limit lower=0 upper=1.677 effort=0 velocity=0 -> lower=0 upper=1.677 effort=27 velocity=1.5
- joint 4-joint: limit (none) -> lower=-1.79677778 upper=1.79677778 effort=27 velocity=1.5; type continuous -> revolute
- joint 5-joint: limit lower=-1.677 upper=0 effort=0 velocity=0 -> lower=-1.677 upper=0 effort=7 velocity=1.5
