Commit message: chore: 零位标定、URDF 限位与 Servo/串口 TX 弧度偏移
- TRoMaC: initial_positions 对齐下位机；joint_limits 收紧速度与加速度
- servo_settings: 降低笛卡尔缩放，JointJog 缩放 0.70
- serial_comm_node: /joint_states 转串口度数前减去 joint_offset_rad（与零位一致）；预留 RX hex 调试块
- manipulator.urdf: 两处关节 limit 与实物一致
- moveit_servo: 奇异 HALT 时保留速度比例 0.05 → 0.02

Made-with: VanNaNY

File: src/manipulator/urdf/manipulator.urdf (robot description, URDF)
Before this commit: robot 机械臂-总装-新-4.SLDASM, 8 links, 7 joints
Joints:
- joint pitch-1-joint: limit lower=-3.1416 upper=0 effort=0 velocity=0 -> lower=-3.1416 upper=-1.7634 effort=0 velocity=0
- joint pitch-3-joint: limit lower=0 upper=4.0942 effort=0 velocity=0 -> lower=0.8066 upper=4.0942 effort=0 velocity=0

Commit message: TRoMaC: 串口回零、笛卡尔前三轴 Jacobian 与 Servo 调参
- serial_comm: 按键 14 触发 HOMING（MoveGroup 规划至 initial_positions）；笛卡尔
  xyz 用前三关节 3×3 阻尼伪逆，六轴统一 JointJog（避免 Twist 抢占）；前三轴组
  按键 13→9；log_auto_send 默认 false，RX 日志可关
- 增加 moveit_ros_planning_interface 依赖
- joint_limits: max_velocity 0.5→0.8；servo scale 线性/旋转/关节→1.0
- moveit.rviz: Planned Path 关闭 Show Robot Visual
- manipulator.urdf: pitch-2-joint 下限调整

Made-with: Cursor

File: src/manipulator/urdf/manipulator.urdf (robot description, URDF)
Before this commit: robot 机械臂-总装-新-4.SLDASM, 8 links, 7 joints
Joints:
- joint pitch-3-joint: limit lower=0.8066 upper=4.0942 effort=0 velocity=0 -> lower=0.470 upper=4.0942 effort=0 velocity=0

Commit message: 改死区和一键动作

File: src/manipulator/urdf/manipulator.urdf (robot description, URDF)
Before this commit: robot manipulator, 7 links, 6 joints
Joints:
- joint 1-joint: limit lower=-2.1765 upper=1.1728 effort=27 velocity=1.5 -> lower=-3.1365 upper=3.1328 effort=27 velocity=1.5

Commit message: 把大pitch固定，变成5轴机械臂，满足限高但不好用

File: src/manipulator/urdf/manipulator.urdf (robot description, URDF)
Before this commit: robot manipulator, 7 links, 6 joints
Joints:
- joint 3-joint: limit lower=0.5236 upper=2.7674 effort=27 velocity=1.5 -> lower=0.7274 upper=3.0774 effort=27 velocity=1.5
- joint 4-joint: limit lower=-4.6562023 upper=-1.09677778 effort=27 velocity=1.5 -> lower=-3.0 upper=3.08 effort=7 velocity=1.5
- joint 5-joint: limit lower=-1.677 upper=0 effort=7 velocity=1.5 -> lower=0.800405 upper=2.4 effort=7 velocity=1.5
