Commit message: chore: 更新机械臂模型与 MoveIt/串口配置，忽略 node_modules
- TRoMaC: 配置与串口、Servo 相关调整
- manipulator: 新网格与 launch，URDF/CMake 同步
- 根目录: .gitignore 增加 node_modules；补充 package.json 与说明文档

Made-with: Cursor

File: src/TRoMaC_2026_Manipulator/config/机械臂-总装-新-4.SLDASM.ros2_control.xacro (robot description, xacro)
@@ -8,43 +8,43 @@
                 <plugin>mock_components/GenericSystem</plugin>
             </hardware>
-            <joint name="yaw-1-joint">
+            <joint name="1-joint">
                 <command_interface name="position"/>
                 <state_interface name="position">
-                  <param name="initial_value">${initial_positions['yaw-1-joint']}</param>
+                  <param name="initial_value">${initial_positions['1-joint']}</param>
                 </state_interface>
                 <state_interface name="velocity"/>
             </joint>
-            <joint name="pitch-1-joint">
+            <joint name="2-joint">
                 <command_interface name="position"/>
                 <state_interface name="position">
-                  <param name="initial_value">${initial_positions['pitch-1-joint']}</param>
+                  <param name="initial_value">${initial_positions['2-joint']}</param>
                 </state_interface>
                 <state_interface name="velocity"/>
             </joint>
-            <joint name="pitch-2-joint">
+            <joint name="3-joint">
                 <command_interface name="position"/>
                 <state_interface name="position">
-                  <param name="initial_value">${initial_positions['pitch-2-joint']}</param>
+                  <param name="initial_value">${initial_positions['3-joint']}</param>
                 </state_interface>
                 <state_interface name="velocity"/>
             </joint>
-            <joint name="roll-1-joint">
+            <joint name="4-joint">
                 <command_interface name="position"/>
                 <state_interface name="position">
-                  <param name="initial_value">${initial_positions['roll-1-joint']}</param>
+                  <param name="initial_value">${initial_positions['4-joint']}</param>
                 </state_interface>
                 <state_interface name="velocity"/>
             </joint>
-            <joint name="pitch-3-joint">
+            <joint name="5-joint">
                 <command_interface name="position"/>
                 <state_interface name="position">
-                  <param name="initial_value">${initial_positions['pitch-3-joint']}</param>
+                  <param name="initial_value">${initial_positions['5-joint']}</param>
                 </state_interface>
                 <state_interface name="velocity"/>
             </joint>
-            <joint name="roll-2-joint">
+            <joint name="6-joint">
                 <command_interface name="position"/>
                 <state_interface name="position">
-                  <param name="initial_value">${initial_positions['roll-2-joint']}</param>
+                  <param name="initial_value">${initial_positions['6-joint']}</param>
                 </state_interface>
                 <state_interface name="velocity"/>

File: src/manipulator/urdf/manipulator.urdf (robot description, URDF)
Before this commit: robot 机械臂-总装-新-4.SLDASM, 8 links, 7 joints
Links:
- removed link base_footprint
- removed link pitch-1_Link
- removed link pitch-2_Link
- removed link pitch-3_Link
- removed link roll-1_Link
- removed link roll-2_Link
- removed link yaw-1_Link
- added link 1_Link, mass 0.572142027172773; collision mesh filename=package://manipulator/meshes/1_Link.STL; visual mesh filename=package://manipulator/meshes/1_Link.STL
- added link 2_Link, mass 0.645668930110417; collision mesh filename=package://manipulator/meshes/2_Link.STL; visual mesh filename=package://manipulator/meshes/2_Link.STL
- added link 3_Link, mass 0.56534838958726; collision mesh filename=package://manipulator/meshes/3_Link.STL; visual mesh filename=package://manipulator/meshes/3_Link.STL
- added link 4_Link, mass 0.153929257708957; collision mesh filename=package://manipulator/meshes/4_Link.STL; visual mesh filename=package://manipulator/meshes/4_Link.STL
- added link 5_Link, mass 0.254987959093994; collision mesh filename=package://manipulator/meshes/5_Link.STL; visual mesh filename=package://manipulator/meshes/5_Link.STL
- added link 6Link, mass 0.0433474772069015; collision mesh filename=package://manipulator/meshes/6Link.STL; visual mesh filename=package://manipulator/meshes/6Link.STL
- link base_link: mass 0.0556763627352784 -> 0.0136482597260318
Joints:
- removed joint base_footprint_joint
- removed joint pitch-1-joint
- removed joint pitch-2-joint
- removed joint pitch-3-joint
- removed joint roll-1-joint
- removed joint roll-2-joint
- removed joint yaw-1-joint
- added joint 1-joint: type continuous, parent base_link, child 1_Link, origin xyz=0 0 0.0025 rpy=0 0 0, axis 0 0 1
- added joint 2-joint: type revolute, parent 1_Link, child 2_Link, origin xyz=0 -0.02455 0.0665000000000001 rpy=0 0 0, axis 0 1 0, limit lower=0 upper=2.6834 effort=0 velocity=0
- added joint 3-joint: type revolute, parent 2_Link, child 3_Link, origin xyz=-0.226380000000001 -0.0835500000000032 0 rpy=0 0 0, axis 0 -1 0, limit lower=0 upper=1.677 effort=0 velocity=0
- added joint 4-joint: type continuous, parent 3_Link, child 4_Link, origin xyz=0.167395812911923 0.0315000000000018 -0.00118398460991795 rpy=0 0 0, axis -0.999974987526421 0 0.00707278739496964
- added joint 5-joint: type revolute, parent 4_Link, child 5_Link, origin xyz=0.0359990995509461 -0.0300000000000021 -0.000254620346217899 rpy=0 0 0, axis 0 -1 0, limit lower=-1.677 upper=0 effort=0 velocity=0
- added joint 6-joint: type continuous, parent 5_Link, child 6Link, origin xyz=0.0943519303016779 0.0310000000000022 -0.0413143225570544 rpy=0 0 0, axis -0.917582028180844 0 0.397546502386234

Commit message: 更新限位后第一版机械臂，写了一键动作

File: src/TRoMaC_2026_Manipulator/config/机械臂-总装-新-4.SLDASM.ros2_control.xacro (robot description, xacro)
@@ -14,11 +14,4 @@
                 <state_interface name="position">
                   <param name="initial_value">${initial_positions['1-joint']}</param>
-                </state_interface>
-                <state_interface name="velocity"/>
-            </joint>
-            <joint name="2-joint">
-                <command_interface name="position"/>
-                <state_interface name="position">
-                  <param name="initial_value">${initial_positions['2-joint']}</param>
                 </state_interface>
                 <state_interface name="velocity"/>

File: src/manipulator/urdf/manipulator.urdf (robot description, URDF)
Before this commit: robot manipulator, 7 links, 6 joints
Joints:
- joint 1-joint: limit lower=-3.1365 upper=3.1328 effort=27 velocity=1.5 -> lower=-3.1365 upper=3.1328 effort=27 velocity=2.5
- joint 2-joint: axis 0 1 0 -> (none); limit lower=0 upper=2.6834 effort=40 velocity=1.5 -> (none); type revolute -> fixed
- joint 3-joint: limit lower=0 upper=1.677 effort=27 velocity=1.5 -> lower=0.5236 upper=2.7674 effort=27 velocity=1.5
- joint 4-joint: limit lower=-1.79677778 upper=1.79677778 effort=27 velocity=1.5 -> lower=-4.6562023 upper=-1.09677778 effort=27 velocity=1.5
